File: templates/arduino-uno-shield/arduino-101.sch (KiCad schematic (older format))
At the start: 8 parts, among them P1 POWER, P2 ANALOG, P3 DIGITAL, P4 DIGITAL

Commit message: Added complete Arduino 101 template with wickerlib features. Ready for use.
Parts:
- removed P1: POWER, Socket_Arduino_Uno:Socket_Strip_Arduino_1x08, symbol CONN_01X08
- removed P2: ANALOG, Socket_Arduino_Uno:Socket_Strip_Arduino_1x06, symbol CONN_01X06
- removed P3: DIGITAL, Socket_Arduino_Uno:Socket_Strip_Arduino_1x10, symbol CONN_01X10
- removed P4: DIGITAL, Socket_Arduino_Uno:Socket_Strip_Arduino_1x08, symbol CONN_01X08
- removed W1, W2, W3, W4: TEST_1P, Socket_Arduino_Uno:Arduino_1pin, symbol TEST_1P
- added U1, U2, U3, U4: HOLE, Wickerlib:ARDUINO-MOUNTING-HOLE, symbol ARDUINO-101-SHIELD
- added U5: ARDUINO-101-SHIELD, Wickerlib:ARDUINO-101-SHIELD, symbol ARDUINO-101-SHIELD
Connections:
- net labels added: A4, A5, D0, D1, D10, D11, D12, D13, D2, D3, D4, D5, D6, D7, D8, D9, RESET, VIN
- net labels removed: 0(Rx), 1(Tx), 10(**/SS), 11(**/MOSI), 12(MISO), 13(SCK), 2, 3(**), 4, 5(**), 6(**), 7, 8, 9(**), A4(SDA), A5(SCL), AREF, Reset, Vin
- wire segments 37 -> 38
- no-connect marks 9 -> 0
Other:
- note added: "Arduino 101 Shield\nMounting Holes"
- note removed: "Holes"
- note removed: "Shield for Arduino that uses\nthe same pin disposition\nlike Arduino 101."
