File: reference-circuits/atmega16u2-breakout/atmega16u2.kicad_pcb (KiCad board)
At the start: 2 copper layers, 68.6 x 53.3 mm, 5 parts, among them U1 HOLE, U2 HOLE, U3 HOLE, U4 HOLE, U5 ARDUINO-101-SHIELD

Commit message: Schematic verified, printed.
Parts:
- removed U1, U2, U3, U4: HOLE, Wickerlib:ARDUINO-MOUNTING-HOLE
- removed U5: ARDUINO-101-SHIELD, Wickerlib:ARDUINO-101-SHIELD
Other:
- board outline removed
