File: templates/atmega328/atmega328.kicad_pcb (KiCad board)
At the start: 2 copper layers, 0 parts

Commit message: Finished Atmega328 template, including board layout.
Parts:
- added C1: 100nF, Wickerlib:0603, F.Cu at (122.2, 104.3)
- added C2: 10uF 25V, Wickerlib:1210, F.Cu at (136.9, 96.0)
- added C3: 22pF, Wickerlib:0603, F.Cu at (117.4, 106.8)
- added C4: 22pF, Wickerlib:0603, F.Cu at (117.5, 116.3)
- added C5: 100nF, Wickerlib:0603, F.Cu at (136.4, 110.7)
- added C6: 10uF 25V, Wickerlib:1210, F.Cu at (110.6, 97.4)
- added C7: 100nF, Wickerlib:0603, F.Cu at (121.9, 109.7)
- added C8: 100nF, Wickerlib:0603, F.Cu at (120.1, 109.7)
- added C9: 100nF, Wickerlib:0603, F.Cu at (136.4, 114.9)
- added D1: 14V, Wickerlib:Diode_SMA, F.Cu at (119.3, 91.4)
- added D2: 20V 1A, Wickerlib:Diode_SMA, F.Cu at (125.5, 89.9)
- added D3: 20V 1A, Wickerlib:Diode_SMA, F.Cu at (116.8, 99.8)
- added F1: 1.1A 25V, Wickerlib:1812, F.Cu at (135.6, 90.0)
- added J1: INPUT, Wickerlib:OSTVN02A150, F.Cu at (113.3, 89.7)
- added J2: FTDI, Wickerlib:Pin_Header_Straight_1x06, F.Cu at (112.0, 117.0)
- added J3: ISP-2560, Wickerlib:Pin_Header_Straight_2x03, F.Cu at (130.9, 121.5)
- added J4: DIGOUT1, Wickerlib:Pin_Header_Straight_1x10, F.Cu at (112.3, 127.8)
- added J5: DIGOUT2, Wickerlib:Pin_Header_Straight_1x10, F.Cu at (135.2, 131.2)
- added LED1: AMBER, Wickerlib:0603, F.Cu at (122.9, 120.4)
- added R1: 10K, Wickerlib:0805, F.Cu at (127.9, 102.9)
- added R2: 1K, Wickerlib:0603, F.Cu at (127.1, 119.5)
- added S1: RESET, Wickerlib:SW-B3U-1000P, F.Cu at (133.6, 104.3)
- added U1: NCP1117-5V, Wickerlib:DPAK, F.Cu at (132.3, 96.6)
- added U2: ATMEGA328, Wickerlib:TQFP-32_7x7mm_Pitch0.8mm, F.Cu at (128.4, 111.2)
- added X1: 16MHz 18pF, Wickerlib:CRYSTAL-CTS-4SMD, F.Cu at (115.2, 108.6)
Routing:
- net +5V: track 0.00 -> 73.5 mm
- net /A7(*): track 0.00 -> 35.7 mm, vias 0 -> 2
- net GND: track 0.00 -> 35.3 mm, vias 0 -> 6
- net /~RESET: track 0.00 -> 35.0 mm, vias 0 -> 1
- net /A6(*): track 0.00 -> 32.6 mm, vias 0 -> 1
- net /A0: track 0.00 -> 31.3 mm, vias 0 -> 3
- net /D2: track 0.00 -> 29.9 mm, vias 0 -> 1
- net /A5: track 0.00 -> 29.3 mm, vias 0 -> 2
- net /A4: track 0.00 -> 28.3 mm, vias 0 -> 2
- net /A1: track 0.00 -> 28.1 mm, vias 0 -> 1
- net /D3: track 0.00 -> 27.8 mm, vias 0 -> 1
- net /D0: track 0.00 -> 27.7 mm, vias 0 -> 1
- net /A2: track 0.00 -> 27.7 mm, vias 0 -> 2
- net /A3: track 0.00 -> 27.6 mm, vias 0 -> 2
- net /D4: track 0.00 -> 26.0 mm, vias 0 -> 1
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- added copper zone on B.Cu, net GND
- added copper zone on F.Cu, net GND
Other:
- board outline added: 35.6 x 48.3 mm
- board text added: "5V"
- board text added: "A0"
- board text added: "A1"
- board text added: "A2"
- board text added: "A3"
- board text added: "A4"
- board text added: "A5"
- board text added: "A6"
- board text added: "A7"
- board text added: "Atmega328 Breakout v1.0"
- board text added: "D10"
- board text added: "D11"
- board text added: "D12"
- board text added: "D13"
- board text added: "D2"
- board text added: "D3"
- board text added: "D4"
- board text added: "D5"
- board text added: "D6"
- board text added: "D7"
- board text added: "D8"
- board text added: "D9"
- board text added: "FTDI"
- board text added: "GND"
- board text added: "NC"
- board text added: "RST"
- board text added: "RX"
- board text added: "TX"
- board text added: "VIN"
- board text added: "wickerbox.net/wickerlib"
