File: templates/atmega328/atmega328.kicad_pcb (KiCad board)
At the start: 2 copper layers, 35.6 x 48.3 mm, 25 parts, among them J1 INPUT, J2 FTDI, J3 ISP-2560, J4 DIGOUT1, J5 DIGOUT2, U1 NCP1117-5V, U2 ATMEGA328, X1 16MHz 18pF

Commit message: Removed implementation and left only the raw template.
Parts:
- removed C1, C5, C7, C8, C9: 100nF, Wickerlib:0603
- removed C2, C6: 10uF 25V, Wickerlib:1210
- removed C3, C4: 22pF, Wickerlib:0603
- removed D1: 14V, Wickerlib:Diode_SMA
- removed D2, D3: 20V 1A, Wickerlib:Diode_SMA
- removed F1: 1.1A 25V, Wickerlib:1812
- removed J1: INPUT, Wickerlib:OSTVN02A150
- removed J2: FTDI, Wickerlib:Pin_Header_Straight_1x06
- removed J3: ISP-2560, Wickerlib:Pin_Header_Straight_2x03
- removed J4: DIGOUT1, Wickerlib:Pin_Header_Straight_1x10
- removed J5: DIGOUT2, Wickerlib:Pin_Header_Straight_1x10
- removed LED1: AMBER, Wickerlib:0603
- removed R1: 10K, Wickerlib:0805
- removed R2: 1K, Wickerlib:0603
- removed S1: RESET, Wickerlib:SW-B3U-1000P
- removed U1: NCP1117-5V, Wickerlib:DPAK
- removed U2: ATMEGA328, Wickerlib:TQFP-32_7x7mm_Pitch0.8mm
- removed X1: 16MHz 18pF, Wickerlib:CRYSTAL-CTS-4SMD
Routing:
- net +5V: track 73.5 -> 0.00 mm
- net /A7(*): track 35.7 -> 0.00 mm, vias 2 -> 0
- net GND: track 35.3 -> 0.00 mm, vias 6 -> 0
- net /~RESET: track 35.0 -> 0.00 mm, vias 1 -> 0
- net /A6(*): track 32.6 -> 0.00 mm, vias 1 -> 0
- net /A0: track 31.3 -> 0.00 mm, vias 3 -> 0
- net /D2: track 29.9 -> 0.00 mm, vias 1 -> 0
- net /A5: track 29.3 -> 0.00 mm, vias 2 -> 0
- net /A4: track 28.3 -> 0.00 mm, vias 2 -> 0
- net /A1: track 28.1 -> 0.00 mm, vias 1 -> 0
- net /D3: track 27.8 -> 0.00 mm, vias 1 -> 0
- net /D0: track 27.7 -> 0.00 mm, vias 1 -> 0
- net /A2: track 27.7 -> 0.00 mm, vias 2 -> 0
- net /A3: track 27.6 -> 0.00 mm, vias 2 -> 0
- net /D4: track 26.0 -> 0.00 mm, vias 1 -> 0
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- removed copper zone on B.Cu, net GND
- removed copper zone on F.Cu, net GND
Other:
- board outline removed
- net class Default: clearance 0.254 -> 0.2; trace_width 0.254 -> 0.25; via_dia 0.6858 -> 0.6; via_drill 0.3302 -> 0.4
- rule pad_to_mask_clearance: 0.2 -> 0.003
- rule trace_clearance: 0.254 -> 0.2
- rule trace_min: 0.1524 -> 0.2
- rule via_min_drill: 0.3302 -> 0.3
- rule via_min_size: 0.6858 -> 0.4
- board text removed: "5V"
- board text removed: "A0"
- board text removed: "A1"
- board text removed: "A2"
- board text removed: "A3"
- board text removed: "A4"
- board text removed: "A5"
- board text removed: "A6"
- board text removed: "A7"
- board text removed: "Atmega328 Breakout v1.0"
- board text removed: "D10"
- board text removed: "D11"
- board text removed: "D12"
- board text removed: "D13"
- board text removed: "D2"
- board text removed: "D3"
- board text removed: "D4"
- board text removed: "D5"
- board text removed: "D6"
- board text removed: "D7"
- board text removed: "D8"
- board text removed: "D9"
- board text removed: "FTDI"
- board text removed: "GND"
- board text removed: "NC"
- board text removed: "RST"
- board text removed: "RX"
- board text removed: "TX"
- board text removed: "VIN"
- board text removed: "wickerbox.net/wickerlib"

Commit message: All templates are updated, new zips are released.
Other:
- rule pad_to_mask_clearance: 0.003 -> 0.0762
- rule solder_mask_min_width: 0.004 -> 0.1016
- rule trace_clearance: 0.2 -> 0.254
- rule trace_min: 0.2 -> 0.1524
- rule via_min_drill: 0.3 -> 0.3302
- rule via_min_size: 0.4 -> 0.6858
Changed lines of the file:
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@@
-(kicad_pcb (version 4) (host pcbnew 4.0.1-3.201512221402+6198~38~ubuntu14.04.1-stable)
+(kicad_pcb (version 4) (host pcbnew 4.0.4+e1-6308~48~ubuntu14.04.1-stable)
   (general
     (links 0)
@@
     (nets 1)
   )
-  (page A4)
+  (page USLetter)
+  (title_block
+    (company "Released under the CERN Open Hardware License v1.2")
+    (comment 1 "jenner@wickerbox.net - http://wickerbox.net")
+    (comment 2 "Designed by Jenner at Wickerbox Electronics")
+  )
   (layers
     (0 F.Cu signal)
@@
     (49 F.Fab user)
   )
+  (layers
+    (0 F.Cu signal)
+    (31 B.Cu signal)
+    (34 B.Paste user)
+    (35 F.Paste user)
+    (36 B.SilkS user)
+    (37 F.SilkS user)
+    (38 B.Mask user)
+    (39 F.Mask user)
+    (44 Edge.Cuts user)
+    (46 B.CrtYd user)
+    (47 F.CrtYd user)
+    (48 B.Fab user)
+    (49 F.Fab user)
+  )
   (setup
-    (last_trace_width 0.25)
-    (trace_clearance 0.2)
+    (last_trace_width 0.254)
+    (user_trace_width 0.1524)
+    (user_trace_width 0.254)
+    (user_trace_width 0.3302)
+    (user_trace_width 0.508)
+    (user_trace_width 0.762)
+    (user_trace_width 1.27)
+    (trace_clearance 0.254)
     (zone_clearance 0.508)
     (zone_45_only no)
-    (trace_min 0.2)
-    (segment_width 0.15)
-    (edge_width 0.1)
-    (via_size 0.6)
-    (via_drill 0.4)
-    (via_min_size 0.4)
-    (via_min_drill 0.3)
-    (uvia_size 0.3)
-    (uvia_drill 0.1)
+    (trace_min 0.1524)
+    (segment_width 0.1524)
+    (edge_width 0.1524)
+    (via_size 0.6858)
+    (via_drill 0.3302)
+    (via_min_size 0.6858)
+    (via_min_drill 0.3302)
+    (user_via 0.6858 0.3302)
+    (user_via 0.762 0.4064)
+    (user_via 0.8636 0.508)
+    (uvia_size 0.6858)
+    (uvia_drill 0.3302)
     (uvias_allowed no)
-    (uvia_min_size 0.2)
-    (uvia_min_drill 0.1)
-    (pcb_text_width 0.15)
-    (pcb_text_size 1 1)
-    (mod_edge_width 0.15)
-    (mod_text_size 1 1)
-    (mod_text_width 0.15)
-    (pad_size 1.7272 1.7272)
-    (pad_drill 1.016)
-    (pad_to_mask_clearance 0.003)
-    (solder_mask_min_width 0.004)
+    (uvia_min_size 0)
+    (uvia_min_drill 0)
+    (pcb_text_width 0.1524)
+    (pcb_text_size 1.016 1.016)
+    (mod_edge_width 0.1524)
+    (mod_text_size 1.016 1.016)
+    (mod_text_width 0.1524)
+    (pad_size 1.524 1.524)
+    (pad_drill 0.762)
+    (pad_to_mask_clearance 0.0762)
+    (solder_mask_min_width 0.1016)
+    (pad_to_paste_clearance -0.0762)
     (aux_axis_origin 0 0)
-    (visible_elements FFFFFF7F)
+    (visible_elements FFFEDF7D)
     (pcbplotparams
-      (layerselection 0x00030_80000001)
-      (usegerberextensions false)
+      (layerselection 0x310fc_80000001)
+      (usegerberextensions true)
       (excludeedgelayer true)
       (linewidth 0.100000)
@@
       (outputformat 1)
       (mirror false)
-      (drillshape 1)
+      (drillshape 0)
       (scaleselection 1)
-      (outputdirectory ""))
+      (outputdirectory gerbers))
   )
   (net 0 "")

Commit message: Created basic ATMEGA328 breakout board
Parts:
- added C1: 100nF, Wickerlib:RLC-0603-SMD, F.Cu at (171.2, 65.3)
- added C3: 22pF, Wickerlib:RLC-0603-SMD, F.Cu at (141.0, 71.1)
- added C4: 22pF, Wickerlib:RLC-0603-SMD, F.Cu at (134.0, 76.5)
- added C5: 100nF, Wickerlib:RLC-0603-SMD, F.Cu at (137.6, 59.3)
- added C7: 100nF, Wickerlib:RLC-0603-SMD, F.Cu at (145.9, 59.2)
- added C8: 100nF, Wickerlib:RLC-0603-SMD, F.Cu at (133.0, 59.3)
- added C9: 100nF, Wickerlib:RLC-0603-SMD, F.Cu at (141.4, 59.2)
- added J2: FTDI, Wickerlib:CONN-HEADER-STRAIGHT-P2.54MM-1x06, F.Cu at (171.2, 57.7)
- added J3: ISP-2560, Wickerlib:CONN-HEADER-STRAIGHT-P2.54MM-2x03, F.Cu at (194.3, 58.9)
- added J4: DIGOUT1, Wickerlib:CONN-HEADER-STRAIGHT-P2.54MM-1x10, F.Cu at (152.1, 107.8)
- added J5: DIGOUT2, Wickerlib:CONN-HEADER-STRAIGHT-P2.54MM-1x10, F.Cu at (201.7, 74.0)
- added LED1: AMBER, Wickerlib:RLC-0603-SMD, F.Cu at (159.4, 113.5)
- added R1: 10K, Wickerlib:RLC-0805-SMD, F.Cu at (181.1, 65.0)
- added R2: 1K, Wickerlib:RLC-0603-SMD, F.Cu at (164.1, 113.5)
- added S1: RESET, Wickerlib:SWITCH-OMRON-MOMENTARY-SMD-B3U-1000P, F.Cu at (176.5, 62.7)
- added U2: ATMEGA328, Wickerlib:TQFP-32-7x7MM-P0.8MM, F.Cu at (166.6, 82.3)
- added X1: 16MHz 18pF, Wickerlib:CRYSTAL-CTS-4SMD, F.Cu at (141.5, 75.8)
Routing:
- net /D11: track 0.00 -> 63.0 mm
- net /D12: track 0.00 -> 59.5 mm, vias 0 -> 1
- net /D13: track 0.00 -> 54.3 mm, vias 0 -> 1
- net /~RESET: track 0.00 -> 45.4 mm, vias 0 -> 1
- net /D2: track 0.00 -> 35.3 mm, vias 0 -> 2
- net /D3: track 0.00 -> 33.0 mm
- net Net-(C4-Pad1): track 0.00 -> 31.8 mm, vias 0 -> 2
- net /D4: track 0.00 -> 31.3 mm
- net /D7: track 0.00 -> 28.6 mm
- net Net-(C3-Pad1): track 0.00 -> 28.0 mm, vias 0 -> 2
- net /D10: track 0.00 -> 23.6 mm
- net /D5: track 0.00 -> 23.4 mm
- net +5V: track 0.00 -> 23.3 mm, vias 0 -> 5
- net /D9: track 0.00 -> 22.9 mm
- net /D6: track 0.00 -> 22.7 mm
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- added copper zone on B.Cu, net +5V
- added copper zone on F.Cu, net GND
Other:
- board outline added: 84.8 x 66.1 mm
- net class Default: clearance 0.2 -> 0.1524; trace_width 0.25 -> 0.1524; via_dia 0.6 -> 0.6858; via_drill 0.4 -> 0.3302
- rule trace_clearance: 0.254 -> 0.1524
