File: templates/wickerbox-2layer/wickerbox-2layer.kicad_pcb (KiCad board)
At the start: 2 copper layers, 0 parts

Commit message: Adjusted Wickerbox-specific templates.
Other:
- rule pad_to_mask_clearance: 0.2 -> 0.0762
Changed lines of the file:
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@@
-(kicad_pcb (version 4) (host pcbnew 4.0.1-3.201512221402+6198~38~ubuntu14.04.1-stable)
+(kicad_pcb (version 4) (host pcbnew 4.0.4+e1-6308~48~ubuntu14.04.1-stable)
   (general
     (links 0)
@@
     (nets 1)
   )
-  (page A4)
+  (page USLetter)
   (title_block
     (company "Released under the CERN Open Hardware License v1.2")
-    (comment 1 "wickerboxen@gmail.com - http://wickerbox.net")
+    (comment 1 "jenner@wickerbox.net - http://wickerbox.net")
     (comment 2 "Designed by Jenner at Wickerbox Electronics")
   )
@@
     (trace_min 0.1524)
     (segment_width 0.2)
-    (edge_width 0.15)
+    (edge_width 0.1524)
     (via_size 0.6858)
     (via_drill 0.3302)
@@
     (pad_size 1.524 1.524)
     (pad_drill 0.762)
-    (pad_to_mask_clearance 0.2)
+    (pad_to_mask_clearance 0.0762)
+    (solder_mask_min_width 0.1016)
     (aux_axis_origin 0 0)
     (visible_elements FFFEDF7D)
     (pcbplotparams
-      (layerselection 0x000fc_80000001)
+      (layerselection 0x310fc_80000001)
       (usegerberextensions true)
       (excludeedgelayer true)
@@
       (drillshape 0)
       (scaleselection 1)
-      (outputdirectory ""))
+      (outputdirectory gerbers))
   )
   (net 0 "")
