File: templates/wickerbox-2layer/wickerbox-2layer.kicad_pcb (KiCad board)
At the start: 2 copper layers, 0 parts

Commit message: Updated template.
Other:
- rule trace_clearance: 0.254 -> 0.1524
Changed lines of the file:
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@@
     (user_trace_width 0.762)
     (user_trace_width 1.27)
-    (trace_clearance 0.254)
+    (trace_clearance 0.1524)
     (zone_clearance 0.508)
     (zone_45_only no)
