File: templates/wickerbox-4layer/wickerbox-4layer.kicad_pcb (KiCad board)
At the start: 2 copper layers, 0 parts

Commit message: Templates might be good.
Other:
- copper layers 2 -> 4
- rule trace_min: 0.1524 -> 0.127
- rule via_min_drill: 0.3302 -> 0.254
- rule via_min_size: 0.6858 -> 0.508
Changed lines of the file:
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@@
   (page A4)
   (title_block
-    (title "Project Title")
+    (company "Released under the CERN Open Hardware License v1.2")
+    (comment 1 "wickerboxen@gmail.com - http://wickerbox.net")
+    (comment 2 "Designed by Jenner at Wickerbox Electronics")
   )
   (layers
     (0 F.Cu signal)
+    (1 In1.Cu signal)
+    (2 In2.Cu signal)
     (31 B.Cu signal)
     (34 B.Paste user)
@@
   (setup
     (last_trace_width 0.254)
-    (user_trace_width 0.1524)
+    (user_trace_width 0.127)
+    (user_trace_width 0.2032)
     (user_trace_width 0.254)
     (user_trace_width 0.3302)
@@
     (zone_clearance 0.508)
     (zone_45_only no)
-    (trace_min 0.1524)
+    (trace_min 0.127)
     (segment_width 0.2)
     (edge_width 0.15)
     (via_size 0.6858)
     (via_drill 0.3302)
-    (via_min_size 0.6858)
-    (via_min_drill 0.3302)
-    (user_via 0.6858 0.3302)
-    (user_via 0.762 0.4064)
-    (user_via 0.8636 0.508)
+    (via_min_size 0.508)
+    (via_min_drill 0.254)
+    (user_via 0.508 0.254)
+    (user_via 0.5842 0.3302)
+    (user_via 0.762 0.508)
     (uvia_size 0.6858)
     (uvia_drill 0.3302)

Commit message: Updated default text sizes in templates.
Other:
- rule pad_to_mask_clearance: 0.2 -> 0.0762
- rule trace_min: 0.127 -> 0.1524
- rule via_min_drill: 0.254 -> 0.3302
- rule via_min_size: 0.508 -> 0.6858
Changed lines of the file:
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@@
-(kicad_pcb (version 4) (host pcbnew 4.0.1-3.201512221402+6198~38~ubuntu14.04.1-stable)
+(kicad_pcb (version 4) (host pcbnew 4.0.4+e1-6308~48~ubuntu14.04.1-stable)
   (general
     (links 0)
@@
     (nets 1)
   )
-  (page A4)
+  (page USLetter)
   (title_block
     (company "Released under the CERN Open Hardware License v1.2")
-    (comment 1 "wickerboxen@gmail.com - http://wickerbox.net")
+    (comment 1 "jenner@wickerbox.net - http://wickerbox.net")
     (comment 2 "Designed by Jenner at Wickerbox Electronics")
   )
@@
   (setup
     (last_trace_width 0.254)
-    (user_trace_width 0.127)
-    (user_trace_width 0.2032)
+    (user_trace_width 0.1524)
     (user_trace_width 0.254)
     (user_trace_width 0.3302)
@@
     (zone_clearance 0.508)
     (zone_45_only no)
-    (trace_min 0.127)
-    (segment_width 0.2)
-    (edge_width 0.15)
+    (trace_min 0.1524)
+    (segment_width 0.1524)
+    (edge_width 0.1524)
     (via_size 0.6858)
     (via_drill 0.3302)
-    (via_min_size 0.508)
-    (via_min_drill 0.254)
-    (user_via 0.508 0.254)
-    (user_via 0.5842 0.3302)
-    (user_via 0.762 0.508)
+    (via_min_size 0.6858)
+    (via_min_drill 0.3302)
+    (user_via 0.6858 0.3302)
+    (user_via 0.762 0.4064)
+    (user_via 0.8636 0.508)
     (uvia_size 0.6858)
     (uvia_drill 0.3302)
@@
     (uvia_min_size 0)
     (uvia_min_drill 0)
-    (pcb_text_width 0.3)
-    (pcb_text_size 1.5 1.5)
-    (mod_edge_width 0.15)
-    (mod_text_size 1 1)
-    (mod_text_width 0.15)
+    (pcb_text_width 0.1524)
+    (pcb_text_size 1.016 1.016)
+    (mod_edge_width 0.1524)
+    (mod_text_size 1.016 1.016)
+    (mod_text_width 0.1524)
     (pad_size 1.524 1.524)
     (pad_drill 0.762)
-    (pad_to_mask_clearance 0.2)
+    (pad_to_mask_clearance 0.0762)
+    (solder_mask_min_width 0.1016)
     (aux_axis_origin 0 0)
     (visible_elements FFFEDF7D)
     (pcbplotparams
-      (layerselection 0x000fc_80000001)
+      (layerselection 0x310fc_80000001)
       (usegerberextensions true)
       (excludeedgelayer true)
@@
       (drillshape 0)
       (scaleselection 1)
-      (outputdirectory ""))
+      (outputdirectory gerbers))
   )
   (net 0 "")
