File: templates/oshpark-2layer/oshpark-2layer.kicad_pcb (KiCad board)
At the start: 2 copper layers, 0 parts

Commit message: Release.
Other:
- rule pad_to_mask_clearance: 0.2 -> 0.0762
Changed lines of the file:
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@@
     (nets 1)
   )
-  (page A4)
+  (page USLetter)
   (title_block
     (title "Project Title")
@@
     (zone_45_only no)
     (trace_min 0.1524)
-    (segment_width 0.2)
-    (edge_width 0.15)
+    (segment_width 0.1524)
+    (edge_width 0.1524)
     (via_size 0.6858)
     (via_drill 0.3302)
@@
     (uvia_min_size 0)
     (uvia_min_drill 0)
-    (pcb_text_width 0.3)
-    (pcb_text_size 1.5 1.5)
-    (mod_edge_width 0.15)
-    (mod_text_size 1 1)
-    (mod_text_width 0.15)
+    (pcb_text_width 0.1524)
+    (pcb_text_size 1.016 1.016)
+    (mod_edge_width 0.1524)
+    (mod_text_size 1.016 1.016)
+    (mod_text_width 0.1524)
     (pad_size 1.524 1.524)
     (pad_drill 0.762)
-    (pad_to_mask_clearance 0.2)
+    (pad_to_mask_clearance 0.0762)
+    (solder_mask_min_width 0.1016)
+    (pad_to_paste_clearance -0.0762)
     (aux_axis_origin 0 0)
     (visible_elements FFFEDF7D)
     (pcbplotparams
-      (layerselection 0x000fc_80000001)
+      (layerselection 0x310fc_80000001)
       (usegerberextensions true)
       (excludeedgelayer true)
@@
       (drillshape 0)
       (scaleselection 1)
-      (outputdirectory ""))
+      (outputdirectory gerbers))
   )
   (net 0 "")
