File: templates/arduino-101-shield/arduino-101.sch (KiCad schematic (older format))
At the start: 5 parts, among them U1 HOLE, U2 HOLE, U3 HOLE, U4 HOLE, U5 ARDUINO-101-SHIELD

Commit message: Releasing Arduino 101 template.
Parts:
- U1, U2, U3, U4: footprint Wickerlib:ARDUINO-MOUNTING-HOLE -> ARDUINO-MOUNTING-HOLE
- U5: footprint Wickerlib:ARDUINO-101-SHIELD -> ARDUINO-101-SHIELD
Connections:
- wire segments 38 -> 39
Changed lines of the file:
@@
 EESchema Schematic File Version 2
-LIBS:wickerlib
 LIBS:arduino-101-cache
 EELAYER 25 0
@@
 F 0 "U1" H 1175 1100 50  0001 L CNN
 F 1 "HOLE" V 1125 1150 50  0001 L CNN
-F 2 "Wickerlib:ARDUINO-MOUNTING-HOLE" H 1325 1250 50  0001 C CIN
+F 2 "ARDUINO-MOUNTING-HOLE" H 1325 1250 50  0001 C CIN
 F 3 "https://www.adafruit.com/products/50" H 1325 1600 10  0001 C CNN
 F 4 "ARDU-101SHIELD" H 1325 1250 50  0001 C CIN "Package"
@@
 F 0 "U2" H 1275 1100 50  0001 L CNN
 F 1 "HOLE" V 1225 1150 50  0001 L CNN
-F 2 "Wickerlib:ARDUINO-MOUNTING-HOLE" H 1425 1250 50  0001 C CIN
+F 2 "ARDUINO-MOUNTING-HOLE" H 1425 1250 50  0001 C CIN
 F 3 "https://www.adafruit.com/products/50" H 1425 1600 5   0001 C CNN
 F 4 "ARDU-101SHIELD" H 1425 1250 50  0001 C CIN "Package"
@@
 F 0 "U3" H 1375 1100 50  0001 L CNN
 F 1 "HOLE" V 1325 1150 50  0001 L CNN
-F 2 "Wickerlib:ARDUINO-MOUNTING-HOLE" H 1525 1250 50  0001 C CIN
+F 2 "ARDUINO-MOUNTING-HOLE" H 1525 1250 50  0001 C CIN
 F 3 "https://www.adafruit.com/products/50" H 1525 1600 5   0001 C CNN
 F 4 "ARDU-101SHIELD" H 1525 1250 50  0001 C CIN "Package"
@@
 F 0 "U4" H 1475 1100 50  0001 L CNN
 F 1 "HOLE" V 1425 1150 50  0001 L CNN
-F 2 "Wickerlib:ARDUINO-MOUNTING-HOLE" H 1625 1250 50  0001 C CIN
+F 2 "ARDUINO-MOUNTING-HOLE" H 1625 1250 50  0001 C CIN
 F 3 "https://www.adafruit.com/products/50" H 1625 1600 5   0001 C CNN
 F 4 "ARDU-101SHIELD" H 1625 1250 50  0001 C CIN "Package"
@@
 	1525 3000 1675 3000
 Wire Wire Line
-	1675 2900 1675 3175
+	1675 2900 1675 3000
+Wire Wire Line
+	1675 3000 1675 3175
 Wire Wire Line
 	1525 2900 1675 2900
@@
 F 0 "U5" H 1225 2250 50  0000 L CNN
 F 1 "ARDUINO-101-SHIELD" V 1175 2300 50  0001 L CNN
-F 2 "Wickerlib:ARDUINO-101-SHIELD" H 1375 2400 50  0001 C CIN
+F 2 "ARDUINO-101-SHIELD" H 1375 2400 50  0001 C CIN
 F 3 "https://www.adafruit.com/products/3033" H 1375 2750 5   0001 C CNN
 F 4 "ARDU-101SHIELD" H 1375 2400 50  0001 C CIN "Package"
@@
 F 0 "U5" H 1225 3150 50  0000 L CNN
 F 1 "ARDUINO-101-SHIELD" V 1175 3200 50  0001 L CNN
-F 2 "Wickerlib:ARDUINO-101-SHIELD" H 1375 3300 50  0001 C CIN
+F 2 "ARDUINO-101-SHIELD" H 1375 3300 50  0001 C CIN
 F 3 "https://www.adafruit.com/products/3033" H 1375 3650 5   0001 C CNN
 F 4 "ARDU-101SHIELD" H 1375 3300 50  0001 C CIN "Package"
@@
 F 0 "U5" H 1225 4250 50  0000 L CNN
 F 1 "ARDUINO-101-SHIELD" V 1175 4300 50  0001 L CNN
-F 2 "Wickerlib:ARDUINO-101-SHIELD" H 1375 4400 50  0001 C CIN
+F 2 "ARDUINO-101-SHIELD" H 1375 4400 50  0001 C CIN
 F 3 "https://www.adafruit.com/products/3033" H 1375 4750 5   0001 C CNN
 F 4 "ARDU-101SHIELD" H 1375 4400 50  0001 C CIN "Package"
@@
 F 0 "U5" H 1225 5525 50  0000 L CNN
 F 1 "ARDUINO-101-SHIELD" V 1175 5575 50  0001 L CNN
-F 2 "Wickerlib:ARDUINO-101-SHIELD" H 1375 5675 50  0001 C CIN
+F 2 "ARDUINO-101-SHIELD" H 1375 5675 50  0001 C CIN
 F 3 "https://www.adafruit.com/products/3033" H 1375 6025 5   0001 C CNN
 F 4 "ARDU-101SHIELD" H 1375 5675 50  0001 C CIN "Package"
