File: templates/atmega2560/atmega2560.kicad_pcb (KiCad board)
At the start: 2 copper layers, 0 parts

Commit message: All templates are updated, new zips are released.
Other:
- rule pad_to_mask_clearance: 0.2 -> 0.0762
Changed lines of the file:
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@@
-(kicad_pcb (version 4) (host pcbnew 4.0.1-3.201512221402+6198~38~ubuntu14.04.1-stable)
+(kicad_pcb (version 4) (host pcbnew 4.0.4+e1-6308~48~ubuntu14.04.1-stable)
   (general
     (links 0)
@@
     (nets 1)
   )
-  (page A4)
+  (page USLetter)
   (title_block
     (title "Atmega2560 KiCad Template")
@@
     (rev v1.0)
     (company "Released under the CERN Open Hardware License v1.2")
-    (comment 1 "wickerboxen@gmail.com - http://wickerbox.net")
+    (comment 1 "jenner@wickerbox.net - http://wickerbox.net")
     (comment 2 "Designed by Jenner at Wickerbox Electronics")
   )
@@
     (39 F.Mask user)
     (44 Edge.Cuts user)
+    (46 B.CrtYd user)
+    (47 F.CrtYd user)
+    (48 B.Fab user)
+    (49 F.Fab user)
   )
   (setup
@@
     (trace_min 0.1524)
     (segment_width 0.1524)
-    (edge_width 0.15)
+    (edge_width 0.1524)
     (via_size 0.6858)
     (via_drill 0.3302)
@@
     (uvia_min_size 0)
     (uvia_min_drill 0)
-    (pcb_text_width 0.3)
-    (pcb_text_size 1.5 1.5)
-    (mod_edge_width 0.15)
-    (mod_text_size 1 1)
-    (mod_text_width 0.15)
+    (pcb_text_width 0.1524)
+    (pcb_text_size 1.016 1.016)
+    (mod_edge_width 0.1524)
+    (mod_text_size 1.016 1.016)
+    (mod_text_width 0.1524)
     (pad_size 1.524 1.524)
     (pad_drill 0.762)
-    (pad_to_mask_clearance 0.2)
-    (aux_axis_origin 124.968 123.825)
-    (grid_origin 131.064 97.536)
-    (visible_elements FFFCDF7D)
+    (pad_to_mask_clearance 0.0762)
+    (solder_mask_min_width 0.1016)
+    (pad_to_paste_clearance -0.0762)
+    (aux_axis_origin 0 0)
+    (visible_elements FFFEDF7D)
     (pcbplotparams
-      (layerselection 0x00030_80000001)
-      (usegerberextensions false)
+      (layerselection 0x310fc_80000001)
+      (usegerberextensions true)
       (excludeedgelayer true)
       (linewidth 0.100000)
@@
       (drillshape 0)
       (scaleselection 1)
-      (outputdirectory ""))
+      (outputdirectory gerbers))
   )
   (net 0 "")
