File: templates/teensy-3.2/teensy-3.2.kicad_pcb (KiCad board)
At the start: 2 copper layers, 1 part, among them J1 TEENSY LC

Commit message: Releasing Teensy 3.2 template.
Parts:
- J1: footprint Wickerlib:TEENSY-LC -> TEENSY-LC
Changed lines of the file:
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@@
   (page A4)
   (title_block
-    (company "This design uses a KiCad DIP template created by Jenner at Wickerbox Electronics")
+    (company "This design uses a KiCad Teensy template created by Jenner at Wickerbox Electronics")
     (comment 1 "Released under the CERN Open Hardware License v1.2")
   )
@@
     (add_net GND)
   )
-  (module Wickerlib:TEENSY-LC (layer F.Cu)
+  (module TEENSY-LC (layer F.Cu)
     (at 105.41 82.804)
     (fp_text reference J1 (at -7.62 20.066 270) (layer F.SilkS)
