File: examples/throwie-layers/throwie-layers.kicad_pcb (KiCad board)
At the start: 2 copper layers, 0 parts

Commit message: Finish Throwie example v1.0.
Parts:
- added BAT1: CR1220, Wickerlib:BATT-HOLDER-CR1220-BK-916, F.Cu at (61.0, 31.5)
- added LED1: RED, Wickerlib:LED-D5MM-2PIN, F.Cu at (61.0, 41.6)
Routing:
- net +3V: track 0.00 -> 33.1 mm
- net GND: track 0.00 -> 10.1 mm
- net (no net): track 0.00 -> 5.72 mm
Other:
- board outline added: 22.9 x 26.7 mm
- rule trace_clearance: 0.1524 -> 0.254
- board text added: "FABRICATION NOTES 1. THIS IS A 2 LAYER BOARD. 2. EXTERNAL LAYERS SHALL HAVE 1 OZ COPPER. 3. MATERIAL: FR4 AND 0.062 INCH +/- 10% THICK. 4. BOARDS SHALL BE ROHS COMPLIANT. 5. MANUFACTURE IN ACCORDANCE WITH IPC-6012 CLASS 2 6. MASK: BOTH SIDES OF THE BOARD SHALL HAVE SOLDER MASK (ANY COLOR) OVER BARE COPPER. 7. SILK: BOTH SIDES OF THE BOARD SHALL HAVE WHITE SILKSCREEN. DO NOT PLACE SILK OVER BARE C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"
- board text added: "Light!"
- board text added: "No Light :("
- board text added: "Throwie v1.0"
